Commit message: update urdf

File: panda.URDF (robot description, URDF)
Before this commit: robot panda, 10 links, 9 joints
Links:
- removed link panda_link0
- removed link panda_link1
- removed link panda_link2
- removed link panda_link3
- removed link panda_link4
- removed link panda_link5
- removed link panda_link6
- removed link panda_link7
- removed link panda_link8
- removed link world
- added link base_link, mass 0.629769; visual mesh filename=link0.stl
- added link link1, mass 4.970684; visual mesh filename=link1.stl
- added link link2, mass 0.646926; visual mesh filename=link2.stl
- added link link3, mass 3.228604; visual mesh filename=link3.stl
- added link link4, mass 3.587895; visual mesh filename=link4.stl
- added link link5, mass 1.225946; visual mesh filename=link5_0.obj; visual mesh filename=link5_1.obj
- added link link6, mass 1.666555; visual mesh filename=link6.stl
- added link link7, mass 0.735522; visual mesh filename=link7.stl
Joints:
- removed joint panda_joint1
- removed joint panda_joint2
- removed joint panda_joint3
- removed joint panda_joint4
- removed joint panda_joint5
- removed joint panda_joint6
- removed joint panda_joint7
- removed joint panda_joint8
- removed joint world_joint
- added joint joint1: type revolute, parent base_link, child link1, origin xyz=0 0 0.333 rpy=0 0 0, axis 0 0 1, limit lower=-2.8973 upper=2.8973 effort=87.0 velocity=2.1750
- added joint joint2: type revolute, parent link1, child link2, origin xyz=0 0 0 rpy=-1.57079632679 0 0, axis 0 0 1, limit lower=-1.7628 upper=1.7628 effort=87.0 velocity=2.1750
- added joint joint3: type revolute, parent link2, child link3, origin xyz=0 -0.316 0 rpy=1.57079632679 0 0, axis 0 0 1, limit lower=-2.8973 upper=2.8973 effort=87.0 velocity=2.1750
- added joint joint4: type revolute, parent link3, child link4, origin xyz=0.0825 0 0 rpy=1.57079632679 0 0, axis 0 0 1, limit lower=-3.0718 upper=0 effort=87.0 velocity=2.1750
- added joint joint5: type revolute, parent link4, child link5, origin xyz=-0.0825 0.384 0 rpy=-1.57079632679 0 0, axis 0 0 1, limit lower=-2.8973 upper=2.8973 effort=12.0 velocity=2.6100
- added joint joint6: type revolute, parent link5, child link6, origin xyz=0 0 0 rpy=1.57079632679 0 0, axis 0 0 1, limit lower=-0.8 upper=3.7525 effort=12.0 velocity=2.6100
- added joint joint7: type revolute, parent link6, child link7, origin xyz=0.088 0 0 rpy=1.57079632679 0 0, axis 0 0 1, limit lower=-2.8973 upper=2.8973 effort=12.0 velocity=2.6100
