Commit message: test_ik able to reach target pos (TODO add end effector urdf and fix joint6 result)

File: franka_emika_panda/panda.URDF (robot description, URDF)
Before this commit: robot panda, 8 links, 7 joints
Links:
- removed link base_link
- added link link0, mass 0.629769; visual mesh filename=link0.stl
Joints:
- joint joint1: parent base_link -> link0
